File: hardware/v1/garage door opener v1.3 2015 07 16.brd (EAGLE design)
At the start: 45.7 x 40.6 mm, 26 parts, among them K1 HE3621, K2 HE3621

Commit message: Changed value of DS18B20 pull up resistor. Change is insignificant and the old part will continue to work.
Parts:
- R9: value 3.3k -> 43.2
Changed lines of the file:
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@@
 <?xml version="1.0" encoding="utf-8"?>
 <!DOCTYPE eagle SYSTEM "eagle.dtd">
-<eagle version="7.3.0">
+<eagle version="7.5.0">
 <drawing>
 <settings>
@@
 <grid distance="0.05" unitdist="inch" unit="inch" style="lines" multiple="1" display="yes" altdistance="0.05" altunitdist="inch" altunit="inch"/>
 <layers>
-<layer number="1" name="Top" color="4" fill="1" visible="yes" active="yes"/>
+<layer number="1" name="Top" color="4" fill="1" visible="no" active="yes"/>
 <layer number="2" name="Route2" color="1" fill="3" visible="no" active="no"/>
 <layer number="3" name="Route3" color="4" fill="3" visible="no" active="no"/>
@@
 <element name="D4" library="SparkFun-LED" package="LED-0603" value="" x="3.175" y="29.21" rot="R90"/>
 <element name="DS18B20" library="Ava" package="DS1820" value="DS18B20TO92" x="2.54" y="7.62" rot="R90"/>
-<element name="R9" library="resistor" package="R0603" value="3.3k" x="12.7" y="20.32" rot="MR90"/>
+<element name="R9" library="resistor" package="R0603" value="43.2" x="12.7" y="20.32" rot="MR90"/>
 </elements>
 <signals>
