File: hardware/v1/garage door opener v1.3 2015 07 16.sch (EAGLE design)
At the start: 26 parts, among them K1 HE3621, K2 HE3621

Commit message: Changed value of DS18B20 pull up resistor. Change is insignificant and the old part will continue to work.
Parts:
- R9: value 3.3k -> 43.2
Changed lines of the file:
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@@
 <?xml version="1.0" encoding="utf-8"?>
 <!DOCTYPE eagle SYSTEM "eagle.dtd">
-<eagle version="7.3.0">
+<eagle version="7.5.0">
 <drawing>
 <settings>
@@
 <part name="DS18B20" library="Ava" deviceset="DS1820" device="TO92" value="DS18B20TO92"/>
 <part name="+3V5" library="supply1" deviceset="+3V3" device=""/>
-<part name="R9" library="resistor" deviceset="R-US_" device="R0603" value="3.3k"/>
+<part name="R9" library="resistor" deviceset="R-US_" device="R0603" value="43.2"/>
 <part name="GND8" library="supply1" deviceset="GND" device=""/>
 </parts>
